Commit message: simulation pt2

File: 3_DOF.urdf (robot description, URDF)
Before this commit: robot 3DOF_Arm, 4 links, 3 joints
Joints:
- joint joint_2: origin xyz=0 0 0.15 rpy=0 0 0 -> xyz=0 0 0.275 rpy=0 0 0
- joint joint_3: origin xyz=0 0 0.125 rpy=0 0 0 -> xyz=0 0 0.3 rpy=0 0 0

Commit message: Arm w sliders

File: 3_DOF.urdf (robot description, URDF)
Before this commit: robot 3DOF_Arm, 4 links, 3 joints
Links:
- removed link link_1
- removed link link_2
- removed link link_3
- added link base_fixed; visual box size=0.01 0.01 0.01
- added link link1, mass 1.0; collision cylinder length=1.0 radius=0.03; visual cylinder length=1.0 radius=0.03
- added link link2, mass 1.0; collision cylinder length=1.0 radius=0.03; visual cylinder length=1.0 radius=0.03
- link base_link: mass 1 -> None; geometry visual box size=0.1 0.1 0.1
Joints:
- removed joint joint_1
- removed joint joint_2
- removed joint joint_3
- added joint base_yaw: type revolute, parent base_fixed, child base_link, origin xyz=0 0 0 rpy=0 0 0, axis 0 0 1, limit lower=-3.14 upper=3.14 effort=1 velocity=1.0
- added joint joint1: type revolute, parent base_link, child link1, origin xyz=0 0 0 rpy=0 0 0, axis 0 1 0, limit lower=-3.14 upper=3.14 effort=1 velocity=2.0
- added joint joint2: type revolute, parent link1, child link2, origin xyz=0 0 1.0 rpy=0 0 0, axis 0 1 0, limit lower=-3.14 upper=3.14 effort=1 velocity=2.0

Commit message: oct 23 2025 last push

File: 3_DOF.urdf (robot description, URDF)
Before this commit: robot three_link_arm, 4 links, 3 joints
Joints:
- joint joint1: axis 0 1 0 -> 1 0 0
- joint joint2: axis 0 1 0 -> 1 0 0

Commit message: x doesnt affect arm

File: 3_DOF.urdf (robot description, URDF)
Before this commit: robot three_link_arm, 4 links, 3 joints
Joints:
- joint joint1: axis 1 0 0 -> 0 1 0

Commit message: Working arm

File: 3_DOF.urdf (robot description, URDF)
Before this commit: robot three_link_arm, 4 links, 3 joints
Links:
- added link end_effector
- added link world
- link base_fixed: mass None -> 0.01; geometry collision box size=0.01 0.01 0.01; visual box size=0.01 0.01 0.01
- link base_link: mass None -> 0.2; geometry collision box size=0.1 0.1 0.1; visual box size=0.1 0.1 0.1
Joints:
- added joint ee_fixed: type fixed, parent link2, child end_effector, origin xyz=0 0 1.0 rpy=0 0 0
- added joint world_to_base: type fixed, parent world, child base_fixed, origin xyz=0 0 0 rpy=0 0 0
- joint base_yaw: limit lower=-3.14 upper=3.14 effort=1 velocity=1.0 -> lower=-3.14 upper=3.14 effort=100 velocity=2
- joint joint1: limit lower=-3.14 upper=3.14 effort=1 velocity=2.0 -> lower=-3.14 upper=3.14 effort=100 velocity=2
- joint joint2: axis 1 0 0 -> 0 1 0; limit lower=-3.14 upper=3.14 effort=1 velocity=2.0 -> lower=-3.14 upper=3.14 effort=100 velocity=2

Commit message: gripper closes

File: 3_DOF.urdf (robot description, URDF)
Before this commit: robot three_link_arm, 6 links, 5 joints
Links:
- added link left_finger, mass 0.01; collision box size=0.02 0.01 0.1; visual box size=0.02 0.01 0.1
- added link right_finger, mass 0.01; collision box size=0.02 0.01 0.1; visual box size=0.02 0.01 0.1
Joints:
- added joint left_finger_joint: type revolute, parent end_effector, child left_finger, origin xyz=0.02 0 0 rpy=0 0 0, axis 0 1 0, limit lower=-0.6 upper=0.0 effort=50 velocity=1.0
- added joint right_finger_joint: type revolute, parent end_effector, child right_finger, origin xyz=-0.02 0 0 rpy=0 0 0, axis 0 -1 0, limit lower=0.0 upper=0.6 effort=50 velocity=1.0

Commit message: aruco one side works

File: 3_DOF.urdf (robot description, URDF)
Before this commit: robot three_link_arm, 8 links, 7 joints
Links:
- removed link left_finger
- removed link right_finger
Joints:
- removed joint left_finger_joint
- removed joint right_finger_joint

Commit message: added robot arm script and changed urdf

File: 3_DOF.urdf (robot description, URDF)
Before this commit: robot three_link_arm, 6 links, 5 joints
Joints:
- joint world_to_base: origin xyz=0 0 0 rpy=0 0 0 -> xyz=0 0 0 rpy=0 1.5708 0

Commit message: last fix maybe

File: 3_DOF.urdf (robot description, URDF)
Before this commit: robot three_link_arm, 6 links, 5 joints
Links:
- removed link base_fixed
- removed link world
- added link turntable, mass 0.2; collision box size=0.1 0.1 0.1; visual box size=0.1 0.1 0.1
- link base_link: mass 0.2 -> 0.01; geometry collision box size=0.01 0.01 0.01; visual box size=0.01 0.01 0.01
Joints:
- removed joint world_to_base
- joint base_yaw: child base_link -> turntable; origin xyz=0 0 0 rpy=0 0 0 -> xyz=0 0 0 rpy=0 1.5708 0; parent base_fixed -> base_link
- joint joint1: parent base_link -> turntable
